File: hardware/imp-watt-meter.brd (EAGLE design)
At the start: 85.9 x 48.5 mm, 76 parts, among them Q2 535-10200-1-ND, U1 LED_DUAL, U2 PHOTOTRANSISTOR0603, U3 ADE7953ACPZLONGPADS, U4 PHOTOTRANSISTOR0603, U5 LED_DUAL

Commit message: updated name of nets to reflect that SPI is used, not i2c
Connections:
- net I2C_CLOCK_1 renamed MOSI
- net I2C_DATA_2 renamed MISO
Changed lines of the file:
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@@
 <?xml version="1.0" encoding="utf-8"?>
 <!DOCTYPE eagle SYSTEM "eagle.dtd">
-<eagle version="7.4.0">
+<eagle version="7.1.0">
 <drawing>
 <settings>
@@
 <contactref element="PAD1" pad="1"/>
 </signal>
-<signal name="I2C_DATA_2">
+<signal name="MISO">
 <contactref element="U$5" pad="PAD14"/>
 <contactref element="R62" pad="1"/>
@@
 <wire x1="23.9522" y1="11.1252" x2="23.9522" y2="10.4902" width="0.2032" layer="1"/>
 </signal>
-<signal name="I2C_CLOCK_1">
+<signal name="MOSI">
 <contactref element="U$5" pad="PAD22"/>
 <contactref element="R61" pad="2"/>
